Commit message: AgF in sim

File: my_assets/agf1/urdf/agf1.urdf (robot description, URDF)
Before this commit: robot agf1, 1 links, 0 joints
Links:
- added link x_table, mass 1.0; collision cylinder length=0.03 radius=0.075; visual mesh filename=../meshes/Agility_Forge_X_axis_Table.obj scale=0.001 0.001 0.001
- link base_link: geometry collision cylinder length=0.03 radius=0.075; visual mesh filename=../meshes/Agility_Forge_Frame.obj scale=0.001 0.001 0.001
Joints:
- added joint x_table_joint: type prismatic, parent base_link, child x_table, origin xyz=0 0 0 rpy=0 0 0, axis 1 0 0, limit lower=-0.5 upper=0.5 effort=1000 velocity=1.0
- added joint y_table_joint: type prismatic, parent base_link, child x_table, origin xyz=0 0 0 rpy=0 0 0, axis 0 1 0, limit lower=-0.3 upper=0.3 effort=1000 velocity=1.0

Commit message: collision mesh bad

File: my_assets/agf1/urdf/agf1.urdf (robot description, URDF)
Before this commit: robot agf1, 2 links, 2 joints
Links:
- added link workpiece, mass 0; visual mesh filename=../meshes/part_afp.obj scale=0.001 0.001 0.001
Joints:
- removed joint y_table_joint
- added joint workpiece_joint: type floating, parent x_table, child workpiece, origin xyz=0 0 0 rpy=0 0 0

Commit message: Mesh and LiDAR working

File: my_assets/agf1/urdf/agf1.urdf (robot description, URDF)
Before this commit: robot agf1, 3 links, 2 joints
Links:
- removed link workpiece
Joints:
- removed joint workpiece_joint
